File: frickelEKG2.sch (KiCad schematic (older format))
At the start: 80 parts, among them M1 ADS1292R-TQFP, M2 STC3100, M3 LTC4080X, P1 CONN_01X02, P2 CONN_01X02, P3 CONN_01X05, P4 CONN_01X06, P5 USB_B, U1 STM32F030K6, U2 LP5907_3.3V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

Commit message: fixed EXTI
Parts:
- removed P2: CONN_01X02, Connect:PINHEAD1-2, symbol CONN_01X02
- added C42: 1N5, Capacitors_SMD:C_0603, symbol C
- added P2: CONN_01X03, Pin_Headers:Pin_Header_Straight_1x03_Pitch2.54mm, symbol CONN_01X03
- added R17: 100k, Resistors_SMD:R_0603, symbol R
- added R18: 0R, Resistors_SMD:R_0603, symbol R
- added R19: 1M, Resistors_SMD:R_0603, symbol R
- added R20: 10k, Resistors_SMD:R_0603, symbol R
Connections:
- net ADS_DRDY: now also U1.9 (ADC1_IN3/USART1_TX/PA3)
- net DVDD: now also C20.1, C21.1, M1.14 (CLKSEL), M1.23 (DVDD)
- net DVDD_IMU: now also R20.1
- net GND: now also U4.11 (FSYNC), U4.9 (AD0)
- net IN_N: now also P2.2 (P2)
- net IN_P: now also P2.1 (P1)
- net MPU_INT: now reaches U1.28 (SPI1_MOSI/I2C1_SMBA/TIM16_BKIN/TIM3_CH2/PB5)
- net MPU_INT: now also U4.12 (INT), R20.2
- net ADS_RST: now reaches U1.6 (WKUP1/RTC_TAMP2/ADC_IN0/USART1_CTS/PA0)
- net ADS_RST: now also M1.15 (~PWDN/RESET)
- net ADS_START: now reaches U1.7 (ADC1_IN1/USART1_RTS/EVENTOUT/PA1)
- net ADS_START: now also M1.16 (START)
- net RLDINV: now reaches M1.28 (RLDINV)
- net RLDINV: now also C42.2, R19.2
- net RLDIN: now reaches M1.29 (RLDIN/RLDREF)
- net RLDIN: now also R17.1
- net RLDOUT: now reaches M1.30 (RLDOUT)
- net RLDOUT: now also R18.1
- new net RLD_DRV: C42.1, P2.3 (P3), R17.2, R18.2, R19.1
- no-connect marks 0 -> 19
Other:
- moved on the sheet: R2
